File: hardware/pcb_designs/controller_kicad/controller_kicad.kicad_sch (KiCad schematic)
At the start: 3 parts, among them J1 STRIP, J2 POW

Commit message: controller PCB finished
Parts:
- added C1: 100u, Capacitor_THT:CP_Radial_D6.3mm_P2.50mm, symbol Device:C_Polarized
- added C3, C4, C5, C6, C7: 1u, Capacitor_SMD:C_0805_2012Metric_Pad1.18x1.45mm_HandSolder, symbol Device:C
- added D1, D2: LED, LED_THT:LED_D3.0mm, symbol Device:LED
- added J10: BUZZER, Connector_Molex:Molex_KK-254_AE-6410-02A_1x02_P2.54mm_Vertical, symbol Connector:Conn_01x02_Pin
- added J3, J4: POW, Connector_PinHeader_2.54mm:PinHeader_1x02_P2.54mm_Vertical, symbol Connector:Conn_01x02_Pin
- added J5: ANALOGS, Connector_PinHeader_2.54mm:PinHeader_1x08_P2.54mm_Vertical, symbol Connector:Conn_01x08_Pin
- added J6: SW0, Connector_Molex:Molex_KK-254_AE-6410-02A_1x02_P2.54mm_Vertical, symbol Connector:Conn_01x02_Pin
- added J7: SW1, Connector_Molex:Molex_KK-254_AE-6410-02A_1x02_P2.54mm_Vertical, symbol Connector:Conn_01x02_Pin
- added J8: SW2, Connector_Molex:Molex_KK-254_AE-6410-02A_1x02_P2.54mm_Vertical, symbol Connector:Conn_01x02_Pin
- added J9: UART, Connector_PinHeader_2.54mm:PinHeader_1x03_P2.54mm_Vertical, symbol Connector:Conn_01x03_Pin
- added Q1: BC547, Package_TO_SOT_THT:TO-92_HandSolder, symbol Transistor_BJT:BC547
- added R1: 330, Resistor_SMD:R_0805_2012Metric_Pad1.20x1.40mm_HandSolder, symbol Device:R
- added R2, R3: 680, Resistor_SMD:R_0805_2012Metric_Pad1.20x1.40mm_HandSolder, symbol Device:R
- added R4: 2k2, Resistor_SMD:R_0805_2012Metric_Pad1.20x1.40mm_HandSolder, symbol Device:R
Connections:
- net +5V: now also C1.1, C3.1, C4.1, D1.2 (A), D2.2 (A), J10.1 (Pin_1), J3.1 (Pin_1), J3.2 (Pin_2)
- net GND: now also C1.2, C3.2, C4.2, C5.2, C6.2, C7.2, J4.1 (Pin_1), J4.2 (Pin_2), J6.2 (Pin_2), J7.2 (Pin_2), J8.2 (Pin_2), J9.3 (Pin_3), Q1.3 (E), R2.2
- net RGB_DATA: now also A1.6 (D3), R1.2; no longer J1.2 (Pin_2)
- net TX: now reaches A1.1 (D1/TX)
- net TX: now also J9.1 (Pin_1)
- net SW0: now reaches A1.10 (D7)
- net SW0: now also C5.1, J6.1 (Pin_1)
- net SW1: now reaches A1.11 (D8)
- net SW1: now also C6.1, J7.1 (Pin_1)
- net SW2: now reaches A1.12 (D9)
- net SW2: now also C7.1, J8.1 (Pin_1)
- net at A1.19 (A0): now also J5.8 (Pin_8)
- net RX: now reaches A1.2 (D0/RX)
- net RX: now also J9.2 (Pin_2)
- net at A1.20 (A1): now also J5.7 (Pin_7)
- net at A1.21 (A2): now also J5.6 (Pin_6)
- net at A1.22 (A3): now also J5.5 (Pin_5)
- net SDA: now reaches A1.23 (A4)
- net SDA: now also J5.4 (Pin_4)
- net SCL: now reaches A1.24 (A5)
- net SCL: now also J5.3 (Pin_3)
- net at A1.25 (A6): now also J5.2 (Pin_2)
- net at A1.26 (A7): now also J5.1 (Pin_1)
- net BUZZER: now reaches A1.8 (D5)
- net BUZZER: now also R4.1
- net MISC_LED: now reaches A1.9 (D6)
- net MISC_LED: now also R3.2
- new net: J1.2 (Pin_2), R1.1
- new net: D1.1 (K), R2.1
- new net: D2.1 (K), R3.1
- new net: Q1.2 (B), R4.2
- new net: J10.2 (Pin_2), Q1.1 (C)
Other:
- note added: "Arduino Nano schematic https://www.arduino.cc/en/uploads/Main/Arduino_Nano-Rev3.2-SCH.pdf"
- note added: "Buttons"
- note added: "Power input"
- note added: "Pull-up por software"
- note added: "To 1st WS2812 RGB module"
- note added: "VUSB line is protected from +5V line"
- company: (none) -> IEEE-ITBA
- title: (none) -> Controlador de DCF, Display Contador Fútbol
- moved on the sheet: A1, J1, J2
